File: gw-r65x1qsbc-proto1.kicad_pcb (KiCad board)
At the start: 2 copper layers, 129.5 x 104.1 mm, 8 parts, among them J2 PORT D, J3 PORT B, J5 GLITCHBUS

Commit message: PROTOTYPE 1
Parts:
- added J1: PORT D, gw_headers:STRAIGHT_2x5_NOSILK, F.Cu at (177.8, 71.1)
- added J4: PORT B, gw_headers:STRAIGHT_2x5_NOSILK, F.Cu at (86.4, 109.2)
- added J6: GLITCHBUS, gw_headers:STRAIGHT_2x20_NOSILK, F.Cu at (139.7, 137.2)
- added REF**: 70MIL_45DRILL_NO_SILKSCREEN, gw_mounting:70MIL_45DRILL_NO_SILKSCREEN, F.Cu at (78.7, 55.9)
- added REF**: 70MIL_45DRILL_NO_SILKSCREEN, gw_mounting:70MIL_45DRILL_NO_SILKSCREEN, F.Cu at (195.6, 66.0)
- added REF**: 70MIL_45DRILL_NO_SILKSCREEN, gw_mounting:70MIL_45DRILL_NO_SILKSCREEN, F.Cu at (94.0, 124.5)
- added REF**: 70MIL_45DRILL_NO_SILKSCREEN, gw_mounting:70MIL_45DRILL_NO_SILKSCREEN, F.Cu at (124.5, 99.1)
- added REF**: 70MIL_45DRILL_NO_SILKSCREEN, gw_mounting:70MIL_45DRILL_NO_SILKSCREEN, F.Cu at (139.7, 116.8)
- added REF**: 70MIL_45DRILL_NO_SILKSCREEN, gw_mounting:70MIL_45DRILL_NO_SILKSCREEN, F.Cu at (144.8, 104.1)
- added REF**: 70MIL_45DRILL_NO_SILKSCREEN, gw_mounting:70MIL_45DRILL_NO_SILKSCREEN, F.Cu at (127.0, 119.4)
- added REF**: 70MIL_45DRILL_NO_SILKSCREEN, gw_mounting:70MIL_45DRILL_NO_SILKSCREEN, F.Cu at (116.8, 101.6)
- added REF**: 70MIL_45DRILL_NO_SILKSCREEN, gw_mounting:70MIL_45DRILL_NO_SILKSCREEN, F.Cu at (116.8, 81.3)
- added REF**: 70MIL_45DRILL_NO_SILKSCREEN, gw_mounting:70MIL_45DRILL_NO_SILKSCREEN, F.Cu at (132.1, 99.1)
- added REF**: 70MIL_45DRILL_NO_SILKSCREEN, gw_mounting:70MIL_45DRILL_NO_SILKSCREEN, F.Cu at (121.9, 94.0)
- added REF**: 70MIL_45DRILL_NO_SILKSCREEN, gw_mounting:70MIL_45DRILL_NO_SILKSCREEN, F.Cu at (139.7, 109.2)
- added REF**: 70MIL_45DRILL_NO_SILKSCREEN, gw_mounting:70MIL_45DRILL_NO_SILKSCREEN, F.Cu at (137.2, 111.8)
- added REF**: 70MIL_45DRILL_NO_SILKSCREEN, gw_mounting:70MIL_45DRILL_NO_SILKSCREEN, F.Cu at (81.3, 127.0)
- added REF**: 70MIL_45DRILL_NO_SILKSCREEN, gw_mounting:70MIL_45DRILL_NO_SILKSCREEN, F.Cu at (129.5, 81.3)
- added REF**: 70MIL_45DRILL_NO_SILKSCREEN, gw_mounting:70MIL_45DRILL_NO_SILKSCREEN, F.Cu at (129.5, 114.3)
- added REF**: 70MIL_45DRILL_NO_SILKSCREEN, gw_mounting:70MIL_45DRILL_NO_SILKSCREEN, F.Cu at (137.2, 106.7)
- added REF**: 70MIL_45DRILL_NO_SILKSCREEN, gw_mounting:70MIL_45DRILL_NO_SILKSCREEN, F.Cu at (137.2, 116.8)
- added REF**: 70MIL_45DRILL_NO_SILKSCREEN, gw_mounting:70MIL_45DRILL_NO_SILKSCREEN, F.Cu at (129.5, 111.8)
- added REF**: 70MIL_45DRILL_NO_SILKSCREEN, gw_mounting:70MIL_45DRILL_NO_SILKSCREEN, F.Cu at (139.7, 111.8)
- added REF**: 70MIL_45DRILL_NO_SILKSCREEN, gw_mounting:70MIL_45DRILL_NO_SILKSCREEN, F.Cu at (137.2, 109.2)
- added REF**: 70MIL_45DRILL_NO_SILKSCREEN, gw_mounting:70MIL_45DRILL_NO_SILKSCREEN, F.Cu at (116.8, 94.0)
- added REF**: 70MIL_45DRILL_NO_SILKSCREEN, gw_mounting:70MIL_45DRILL_NO_SILKSCREEN, F.Cu at (137.2, 114.3)
- added REF**: 70MIL_45DRILL_NO_SILKSCREEN, gw_mounting:70MIL_45DRILL_NO_SILKSCREEN, F.Cu at (116.8, 116.8)
- added REF**: 70MIL_45DRILL_NO_SILKSCREEN, gw_mounting:70MIL_45DRILL_NO_SILKSCREEN, F.Cu at (81.3, 124.5)
- added REF**: 70MIL_45DRILL_NO_SILKSCREEN, gw_mounting:70MIL_45DRILL_NO_SILKSCREEN, F.Cu at (119.4, 96.5)
- added REF**: 70MIL_45DRILL_NO_SILKSCREEN, gw_mounting:70MIL_45DRILL_NO_SILKSCREEN, F.Cu at (116.8, 99.1)
- added REF**: 70MIL_45DRILL_NO_SILKSCREEN, gw_mounting:70MIL_45DRILL_NO_SILKSCREEN, F.Cu at (119.4, 83.8)
- added REF**: 70MIL_45DRILL_NO_SILKSCREEN, gw_mounting:70MIL_45DRILL_NO_SILKSCREEN, F.Cu at (121.9, 106.7)
- added REF**: 70MIL_45DRILL_NO_SILKSCREEN, gw_mounting:70MIL_45DRILL_NO_SILKSCREEN, F.Cu at (134.6, 106.7)
- added REF**: 70MIL_45DRILL_NO_SILKSCREEN, gw_mounting:70MIL_45DRILL_NO_SILKSCREEN, F.Cu at (132.1, 104.1)
- added REF**: 70MIL_45DRILL_NO_SILKSCREEN, gw_mounting:70MIL_45DRILL_NO_SILKSCREEN, F.Cu at (121.9, 81.3)
- added REF**: 70MIL_45DRILL_NO_SILKSCREEN, gw_mounting:70MIL_45DRILL_NO_SILKSCREEN, F.Cu at (134.6, 104.1)
- added REF**: 70MIL_45DRILL_NO_SILKSCREEN, gw_mounting:70MIL_45DRILL_NO_SILKSCREEN, F.Cu at (127.0, 106.7)
- added REF**: 70MIL_45DRILL_NO_SILKSCREEN, gw_mounting:70MIL_45DRILL_NO_SILKSCREEN, F.Cu at (127.0, 116.8)
- added REF**: 70MIL_45DRILL_NO_SILKSCREEN, gw_mounting:70MIL_45DRILL_NO_SILKSCREEN, F.Cu at (81.3, 129.5)
- added REF**: 70MIL_45DRILL_NO_SILKSCREEN, gw_mounting:70MIL_45DRILL_NO_SILKSCREEN, F.Cu at (127.0, 86.4)
- added REF**: 70MIL_45DRILL_NO_SILKSCREEN, gw_mounting:70MIL_45DRILL_NO_SILKSCREEN, F.Cu at (127.0, 96.5)
- added REF**: 70MIL_45DRILL_NO_SILKSCREEN, gw_mounting:70MIL_45DRILL_NO_SILKSCREEN, F.Cu at (127.0, 91.4)
- added REF**: 70MIL_45DRILL_NO_SILKSCREEN, gw_mounting:70MIL_45DRILL_NO_SILKSCREEN, F.Cu at (129.5, 91.4)
- added REF**: 70MIL_45DRILL_NO_SILKSCREEN, gw_mounting:70MIL_45DRILL_NO_SILKSCREEN, F.Cu at (129.5, 88.9)
- added REF**: 70MIL_45DRILL_NO_SILKSCREEN, gw_mounting:70MIL_45DRILL_NO_SILKSCREEN, F.Cu at (129.5, 86.4)
- added REF**: 70MIL_45DRILL_NO_SILKSCREEN, gw_mounting:70MIL_45DRILL_NO_SILKSCREEN, F.Cu at (127.0, 88.9)
- added REF**: 70MIL_45DRILL_NO_SILKSCREEN, gw_mounting:70MIL_45DRILL_NO_SILKSCREEN, F.Cu at (129.5, 94.0)
- added REF**: 70MIL_45DRILL_NO_SILKSCREEN, gw_mounting:70MIL_45DRILL_NO_SILKSCREEN, F.Cu at (134.6, 111.8)
- added REF**: 70MIL_45DRILL_NO_SILKSCREEN, gw_mounting:70MIL_45DRILL_NO_SILKSCREEN, F.Cu at (132.1, 109.2)
- added REF**: 70MIL_45DRILL_NO_SILKSCREEN, gw_mounting:70MIL_45DRILL_NO_SILKSCREEN, F.Cu at (94.0, 127.0)
- added REF**: 70MIL_45DRILL_NO_SILKSCREEN, gw_mounting:70MIL_45DRILL_NO_SILKSCREEN, F.Cu at (134.6, 109.2)
- added REF**: 70MIL_45DRILL_NO_SILKSCREEN, gw_mounting:70MIL_45DRILL_NO_SILKSCREEN, F.Cu at (132.1, 111.8)
- added REF**: 70MIL_45DRILL_NO_SILKSCREEN, gw_mounting:70MIL_45DRILL_NO_SILKSCREEN, F.Cu at (127.0, 99.1)
- added REF**: 70MIL_45DRILL_NO_SILKSCREEN, gw_mounting:70MIL_45DRILL_NO_SILKSCREEN, F.Cu at (129.5, 83.8)
- added REF**: 70MIL_45DRILL_NO_SILKSCREEN, gw_mounting:70MIL_45DRILL_NO_SILKSCREEN, F.Cu at (132.1, 106.7)
- added REF**: 70MIL_45DRILL_NO_SILKSCREEN, gw_mounting:70MIL_45DRILL_NO_SILKSCREEN, F.Cu at (132.1, 96.5)
- added REF**: 70MIL_45DRILL_NO_SILKSCREEN, gw_mounting:70MIL_45DRILL_NO_SILKSCREEN, F.Cu at (149.9, 114.3)
- added REF**: 70MIL_45DRILL_NO_SILKSCREEN, gw_mounting:70MIL_45DRILL_NO_SILKSCREEN, F.Cu at (149.9, 121.9)
- added REF**: 70MIL_45DRILL_NO_SILKSCREEN, gw_mounting:70MIL_45DRILL_NO_SILKSCREEN, F.Cu at (147.3, 119.4)
- added REF**: 70MIL_45DRILL_NO_SILKSCREEN, gw_mounting:70MIL_45DRILL_NO_SILKSCREEN, F.Cu at (142.2, 94.0)
- added REF**: 70MIL_45DRILL_NO_SILKSCREEN, gw_mounting:70MIL_45DRILL_NO_SILKSCREEN, F.Cu at (96.5, 124.5)
- added REF**: 70MIL_45DRILL_NO_SILKSCREEN, gw_mounting:70MIL_45DRILL_NO_SILKSCREEN, F.Cu at (144.8, 96.5)
- added REF**: 70MIL_45DRILL_NO_SILKSCREEN, gw_mounting:70MIL_45DRILL_NO_SILKSCREEN, F.Cu at (142.2, 99.1)
- added REF**: 70MIL_45DRILL_NO_SILKSCREEN, gw_mounting:70MIL_45DRILL_NO_SILKSCREEN, F.Cu at (139.7, 81.3)
- added REF**: 70MIL_45DRILL_NO_SILKSCREEN, gw_mounting:70MIL_45DRILL_NO_SILKSCREEN, F.Cu at (137.2, 83.8)
- added REF**: 70MIL_45DRILL_NO_SILKSCREEN, gw_mounting:70MIL_45DRILL_NO_SILKSCREEN, F.Cu at (139.7, 101.6)
- added REF**: 70MIL_45DRILL_NO_SILKSCREEN, gw_mounting:70MIL_45DRILL_NO_SILKSCREEN, F.Cu at (144.8, 83.8)
- added REF**: 70MIL_45DRILL_NO_SILKSCREEN, gw_mounting:70MIL_45DRILL_NO_SILKSCREEN, F.Cu at (144.8, 101.6)
- added REF**: 70MIL_45DRILL_NO_SILKSCREEN, gw_mounting:70MIL_45DRILL_NO_SILKSCREEN, F.Cu at (142.2, 101.6)
- added REF**: 70MIL_45DRILL_NO_SILKSCREEN, gw_mounting:70MIL_45DRILL_NO_SILKSCREEN, F.Cu at (144.8, 99.1)
- added REF**: 70MIL_45DRILL_NO_SILKSCREEN, gw_mounting:70MIL_45DRILL_NO_SILKSCREEN, F.Cu at (137.2, 81.3)
- added REF**: 70MIL_45DRILL_NO_SILKSCREEN, gw_mounting:70MIL_45DRILL_NO_SILKSCREEN, F.Cu at (86.4, 124.5)
- added REF**: 70MIL_45DRILL_NO_SILKSCREEN, gw_mounting:70MIL_45DRILL_NO_SILKSCREEN, F.Cu at (137.2, 101.6)
- added REF**: 70MIL_45DRILL_NO_SILKSCREEN, gw_mounting:70MIL_45DRILL_NO_SILKSCREEN, F.Cu at (137.2, 94.0)
- added REF**: 70MIL_45DRILL_NO_SILKSCREEN, gw_mounting:70MIL_45DRILL_NO_SILKSCREEN, F.Cu at (139.7, 96.5)
- added REF**: 70MIL_45DRILL_NO_SILKSCREEN, gw_mounting:70MIL_45DRILL_NO_SILKSCREEN, F.Cu at (137.2, 99.1)
- added REF**: 70MIL_45DRILL_NO_SILKSCREEN, gw_mounting:70MIL_45DRILL_NO_SILKSCREEN, F.Cu at (139.7, 83.8)
- added REF**: 70MIL_45DRILL_NO_SILKSCREEN, gw_mounting:70MIL_45DRILL_NO_SILKSCREEN, F.Cu at (142.2, 106.7)
- added REF**: 70MIL_45DRILL_NO_SILKSCREEN, gw_mounting:70MIL_45DRILL_NO_SILKSCREEN, F.Cu at (154.9, 106.7)
- added REF**: 70MIL_45DRILL_NO_SILKSCREEN, gw_mounting:70MIL_45DRILL_NO_SILKSCREEN, F.Cu at (152.4, 104.1)
- added REF**: 70MIL_45DRILL_NO_SILKSCREEN, gw_mounting:70MIL_45DRILL_NO_SILKSCREEN, F.Cu at (129.5, 96.5)
- added REF**: 70MIL_45DRILL_NO_SILKSCREEN, gw_mounting:70MIL_45DRILL_NO_SILKSCREEN, F.Cu at (132.1, 86.4)
- added REF**: 70MIL_45DRILL_NO_SILKSCREEN, gw_mounting:70MIL_45DRILL_NO_SILKSCREEN, F.Cu at (91.4, 144.8)
- added REF**: 70MIL_45DRILL_NO_SILKSCREEN, gw_mounting:70MIL_45DRILL_NO_SILKSCREEN, F.Cu at (134.6, 86.4)
- added REF**: 70MIL_45DRILL_NO_SILKSCREEN, gw_mounting:70MIL_45DRILL_NO_SILKSCREEN, F.Cu at (142.2, 81.3)
- added REF**: 70MIL_45DRILL_NO_SILKSCREEN, gw_mounting:70MIL_45DRILL_NO_SILKSCREEN, F.Cu at (154.9, 104.1)
- added REF**: 70MIL_45DRILL_NO_SILKSCREEN, gw_mounting:70MIL_45DRILL_NO_SILKSCREEN, F.Cu at (144.8, 86.4)
- added REF**: 70MIL_45DRILL_NO_SILKSCREEN, gw_mounting:70MIL_45DRILL_NO_SILKSCREEN, F.Cu at (144.8, 81.3)
- added REF**: 70MIL_45DRILL_NO_SILKSCREEN, gw_mounting:70MIL_45DRILL_NO_SILKSCREEN, F.Cu at (142.2, 83.8)
- added REF**: 70MIL_45DRILL_NO_SILKSCREEN, gw_mounting:70MIL_45DRILL_NO_SILKSCREEN, F.Cu at (142.2, 96.5)
- added REF**: 70MIL_45DRILL_NO_SILKSCREEN, gw_mounting:70MIL_45DRILL_NO_SILKSCREEN, F.Cu at (139.7, 99.1)
- added REF**: 70MIL_45DRILL_NO_SILKSCREEN, gw_mounting:70MIL_45DRILL_NO_SILKSCREEN, F.Cu at (144.8, 88.9)
- added REF**: 70MIL_45DRILL_NO_SILKSCREEN, gw_mounting:70MIL_45DRILL_NO_SILKSCREEN, F.Cu at (142.2, 86.4)
- added REF**: 70MIL_45DRILL_NO_SILKSCREEN, gw_mounting:70MIL_45DRILL_NO_SILKSCREEN, F.Cu at (88.9, 142.2)
- added REF**: 70MIL_45DRILL_NO_SILKSCREEN, gw_mounting:70MIL_45DRILL_NO_SILKSCREEN, F.Cu at (129.5, 99.1)
- added REF**: 70MIL_45DRILL_NO_SILKSCREEN, gw_mounting:70MIL_45DRILL_NO_SILKSCREEN, F.Cu at (134.6, 88.9)
- added REF**: 70MIL_45DRILL_NO_SILKSCREEN, gw_mounting:70MIL_45DRILL_NO_SILKSCREEN, F.Cu at (149.9, 111.8)
- added REF**: 70MIL_45DRILL_NO_SILKSCREEN, gw_mounting:70MIL_45DRILL_NO_SILKSCREEN, F.Cu at (147.3, 109.2)
- added REF**: 70MIL_45DRILL_NO_SILKSCREEN, gw_mounting:70MIL_45DRILL_NO_SILKSCREEN, F.Cu at (149.9, 109.2)
- added REF**: 70MIL_45DRILL_NO_SILKSCREEN, gw_mounting:70MIL_45DRILL_NO_SILKSCREEN, F.Cu at (147.3, 111.8)
- added REF**: 70MIL_45DRILL_NO_SILKSCREEN, gw_mounting:70MIL_45DRILL_NO_SILKSCREEN, F.Cu at (149.9, 116.8)
- added REF**: 70MIL_45DRILL_NO_SILKSCREEN, gw_mounting:70MIL_45DRILL_NO_SILKSCREEN, F.Cu at (147.3, 114.3)
- added REF**: 70MIL_45DRILL_NO_SILKSCREEN, gw_mounting:70MIL_45DRILL_NO_SILKSCREEN, F.Cu at (152.4, 81.3)
- added REF**: 70MIL_45DRILL_NO_SILKSCREEN, gw_mounting:70MIL_45DRILL_NO_SILKSCREEN, F.Cu at (154.9, 81.3)
- added REF**: 70MIL_45DRILL_NO_SILKSCREEN, gw_mounting:70MIL_45DRILL_NO_SILKSCREEN, F.Cu at (91.4, 142.2)
- added REF**: 70MIL_45DRILL_NO_SILKSCREEN, gw_mounting:70MIL_45DRILL_NO_SILKSCREEN, F.Cu at (152.4, 83.8)
- added REF**: 70MIL_45DRILL_NO_SILKSCREEN, gw_mounting:70MIL_45DRILL_NO_SILKSCREEN, F.Cu at (152.4, 94.0)
- added REF**: 70MIL_45DRILL_NO_SILKSCREEN, gw_mounting:70MIL_45DRILL_NO_SILKSCREEN, F.Cu at (154.9, 96.5)
- added REF**: 70MIL_45DRILL_NO_SILKSCREEN, gw_mounting:70MIL_45DRILL_NO_SILKSCREEN, F.Cu at (152.4, 99.1)
- added REF**: 70MIL_45DRILL_NO_SILKSCREEN, gw_mounting:70MIL_45DRILL_NO_SILKSCREEN, F.Cu at (149.9, 81.3)
- added REF**: 70MIL_45DRILL_NO_SILKSCREEN, gw_mounting:70MIL_45DRILL_NO_SILKSCREEN, F.Cu at (147.3, 83.8)
- added REF**: 70MIL_45DRILL_NO_SILKSCREEN, gw_mounting:70MIL_45DRILL_NO_SILKSCREEN, F.Cu at (149.9, 101.6)
- added REF**: 70MIL_45DRILL_NO_SILKSCREEN, gw_mounting:70MIL_45DRILL_NO_SILKSCREEN, F.Cu at (154.9, 83.8)
- added REF**: 70MIL_45DRILL_NO_SILKSCREEN, gw_mounting:70MIL_45DRILL_NO_SILKSCREEN, F.Cu at (154.9, 101.6)
- added REF**: 70MIL_45DRILL_NO_SILKSCREEN, gw_mounting:70MIL_45DRILL_NO_SILKSCREEN, F.Cu at (152.4, 101.6)
- added REF**: 70MIL_45DRILL_NO_SILKSCREEN, gw_mounting:70MIL_45DRILL_NO_SILKSCREEN, F.Cu at (193.0, 78.7)
- added REF**: 70MIL_45DRILL_NO_SILKSCREEN, gw_mounting:70MIL_45DRILL_NO_SILKSCREEN, F.Cu at (88.9, 144.8)
- added REF**: 70MIL_45DRILL_NO_SILKSCREEN, gw_mounting:70MIL_45DRILL_NO_SILKSCREEN, F.Cu at (154.9, 99.1)
- added REF**: 70MIL_45DRILL_NO_SILKSCREEN, gw_mounting:70MIL_45DRILL_NO_SILKSCREEN, F.Cu at (147.3, 81.3)
- added REF**: 70MIL_45DRILL_NO_SILKSCREEN, gw_mounting:70MIL_45DRILL_NO_SILKSCREEN, F.Cu at (139.7, 106.7)
- added REF**: 70MIL_45DRILL_NO_SILKSCREEN, gw_mounting:70MIL_45DRILL_NO_SILKSCREEN, F.Cu at (137.2, 104.1)
- added REF**: 70MIL_45DRILL_NO_SILKSCREEN, gw_mounting:70MIL_45DRILL_NO_SILKSCREEN, F.Cu at (139.7, 104.1)
- added REF**: 70MIL_45DRILL_NO_SILKSCREEN, gw_mounting:70MIL_45DRILL_NO_SILKSCREEN, F.Cu at (142.2, 116.8)
- added REF**: 70MIL_45DRILL_NO_SILKSCREEN, gw_mounting:70MIL_45DRILL_NO_SILKSCREEN, F.Cu at (132.1, 88.9)
- added REF**: 70MIL_45DRILL_NO_SILKSCREEN, gw_mounting:70MIL_45DRILL_NO_SILKSCREEN, F.Cu at (134.6, 94.0)
- added REF**: 70MIL_45DRILL_NO_SILKSCREEN, gw_mounting:70MIL_45DRILL_NO_SILKSCREEN, F.Cu at (132.1, 91.4)
- added REF**: 70MIL_45DRILL_NO_SILKSCREEN, gw_mounting:70MIL_45DRILL_NO_SILKSCREEN, F.Cu at (147.3, 101.6)
- added REF**: 70MIL_45DRILL_NO_SILKSCREEN, gw_mounting:70MIL_45DRILL_NO_SILKSCREEN, F.Cu at (86.4, 144.8)
- added REF**: 70MIL_45DRILL_NO_SILKSCREEN, gw_mounting:70MIL_45DRILL_NO_SILKSCREEN, F.Cu at (147.3, 94.0)
- added REF**: 70MIL_45DRILL_NO_SILKSCREEN, gw_mounting:70MIL_45DRILL_NO_SILKSCREEN, F.Cu at (149.9, 96.5)
- added REF**: 70MIL_45DRILL_NO_SILKSCREEN, gw_mounting:70MIL_45DRILL_NO_SILKSCREEN, F.Cu at (147.3, 99.1)
- added REF**: 70MIL_45DRILL_NO_SILKSCREEN, gw_mounting:70MIL_45DRILL_NO_SILKSCREEN, F.Cu at (149.9, 83.8)
- added REF**: 70MIL_45DRILL_NO_SILKSCREEN, gw_mounting:70MIL_45DRILL_NO_SILKSCREEN, F.Cu at (152.4, 106.7)
- added REF**: 70MIL_45DRILL_NO_SILKSCREEN, gw_mounting:70MIL_45DRILL_NO_SILKSCREEN, F.Cu at (152.4, 96.5)
- added REF**: 70MIL_45DRILL_NO_SILKSCREEN, gw_mounting:70MIL_45DRILL_NO_SILKSCREEN, F.Cu at (149.9, 99.1)
- added REF**: 70MIL_45DRILL_NO_SILKSCREEN, gw_mounting:70MIL_45DRILL_NO_SILKSCREEN, F.Cu at (154.9, 88.9)
- added REF**: 70MIL_45DRILL_NO_SILKSCREEN, gw_mounting:70MIL_45DRILL_NO_SILKSCREEN, F.Cu at (152.4, 86.4)
- added REF**: 70MIL_45DRILL_NO_SILKSCREEN, gw_mounting:70MIL_45DRILL_NO_SILKSCREEN, F.Cu at (154.9, 86.4)
- added REF**: 70MIL_45DRILL_NO_SILKSCREEN, gw_mounting:70MIL_45DRILL_NO_SILKSCREEN, F.Cu at (91.4, 139.7)
- added REF**: 70MIL_45DRILL_NO_SILKSCREEN, gw_mounting:70MIL_45DRILL_NO_SILKSCREEN, F.Cu at (152.4, 88.9)
- added REF**: 70MIL_45DRILL_NO_SILKSCREEN, gw_mounting:70MIL_45DRILL_NO_SILKSCREEN, F.Cu at (154.9, 94.0)
- added REF**: 70MIL_45DRILL_NO_SILKSCREEN, gw_mounting:70MIL_45DRILL_NO_SILKSCREEN, F.Cu at (152.4, 91.4)
- added REF**: 70MIL_45DRILL_NO_SILKSCREEN, gw_mounting:70MIL_45DRILL_NO_SILKSCREEN, F.Cu at (154.9, 91.4)
- added REF**: 70MIL_45DRILL_NO_SILKSCREEN, gw_mounting:70MIL_45DRILL_NO_SILKSCREEN, F.Cu at (149.9, 119.4)
- added REF**: 70MIL_45DRILL_NO_SILKSCREEN, gw_mounting:70MIL_45DRILL_NO_SILKSCREEN, F.Cu at (147.3, 121.9)
- added REF**: 70MIL_45DRILL_NO_SILKSCREEN, gw_mounting:70MIL_45DRILL_NO_SILKSCREEN, F.Cu at (149.9, 106.7)
- added REF**: 70MIL_45DRILL_NO_SILKSCREEN, gw_mounting:70MIL_45DRILL_NO_SILKSCREEN, F.Cu at (147.3, 104.1)
- added REF**: 70MIL_45DRILL_NO_SILKSCREEN, gw_mounting:70MIL_45DRILL_NO_SILKSCREEN, F.Cu at (149.9, 104.1)
- added REF**: 70MIL_45DRILL_NO_SILKSCREEN, gw_mounting:70MIL_45DRILL_NO_SILKSCREEN, F.Cu at (134.6, 91.4)
- added REF**: 70MIL_45DRILL_NO_SILKSCREEN, gw_mounting:70MIL_45DRILL_NO_SILKSCREEN, F.Cu at (83.8, 142.2)
- added REF**: 70MIL_45DRILL_NO_SILKSCREEN, gw_mounting:70MIL_45DRILL_NO_SILKSCREEN, F.Cu at (129.5, 119.4)
- added REF**: 70MIL_45DRILL_NO_SILKSCREEN, gw_mounting:70MIL_45DRILL_NO_SILKSCREEN, F.Cu at (127.0, 121.9)
- added REF**: 70MIL_45DRILL_NO_SILKSCREEN, gw_mounting:70MIL_45DRILL_NO_SILKSCREEN, F.Cu at (129.5, 106.7)
- added REF**: 70MIL_45DRILL_NO_SILKSCREEN, gw_mounting:70MIL_45DRILL_NO_SILKSCREEN, F.Cu at (127.0, 104.1)
- added REF**: 70MIL_45DRILL_NO_SILKSCREEN, gw_mounting:70MIL_45DRILL_NO_SILKSCREEN, F.Cu at (129.5, 104.1)
- added REF**: 70MIL_45DRILL_NO_SILKSCREEN, gw_mounting:70MIL_45DRILL_NO_SILKSCREEN, F.Cu at (132.1, 116.8)
- added REF**: 70MIL_45DRILL_NO_SILKSCREEN, gw_mounting:70MIL_45DRILL_NO_SILKSCREEN, F.Cu at (121.9, 88.9)
- added REF**: 70MIL_45DRILL_NO_SILKSCREEN, gw_mounting:70MIL_45DRILL_NO_SILKSCREEN, F.Cu at (124.5, 94.0)
- added REF**: 70MIL_45DRILL_NO_SILKSCREEN, gw_mounting:70MIL_45DRILL_NO_SILKSCREEN, F.Cu at (121.9, 91.4)
- added REF**: 70MIL_45DRILL_NO_SILKSCREEN, gw_mounting:70MIL_45DRILL_NO_SILKSCREEN, F.Cu at (119.4, 119.4)
- added REF**: 70MIL_45DRILL_NO_SILKSCREEN, gw_mounting:70MIL_45DRILL_NO_SILKSCREEN, F.Cu at (96.5, 144.8)
- added REF**: 70MIL_45DRILL_NO_SILKSCREEN, gw_mounting:70MIL_45DRILL_NO_SILKSCREEN, F.Cu at (124.5, 91.4)
- added REF**: 70MIL_45DRILL_NO_SILKSCREEN, gw_mounting:70MIL_45DRILL_NO_SILKSCREEN, F.Cu at (116.8, 121.9)
- added REF**: 70MIL_45DRILL_NO_SILKSCREEN, gw_mounting:70MIL_45DRILL_NO_SILKSCREEN, F.Cu at (152.4, 116.8)
- added REF**: 70MIL_45DRILL_NO_SILKSCREEN, gw_mounting:70MIL_45DRILL_NO_SILKSCREEN, F.Cu at (142.2, 88.9)
- added REF**: 70MIL_45DRILL_NO_SILKSCREEN, gw_mounting:70MIL_45DRILL_NO_SILKSCREEN, F.Cu at (144.8, 94.0)
- added REF**: 70MIL_45DRILL_NO_SILKSCREEN, gw_mounting:70MIL_45DRILL_NO_SILKSCREEN, F.Cu at (142.2, 91.4)
- added REF**: 70MIL_45DRILL_NO_SILKSCREEN, gw_mounting:70MIL_45DRILL_NO_SILKSCREEN, F.Cu at (139.7, 119.4)
- added REF**: 70MIL_45DRILL_NO_SILKSCREEN, gw_mounting:70MIL_45DRILL_NO_SILKSCREEN, F.Cu at (144.8, 91.4)
- added REF**: 70MIL_45DRILL_NO_SILKSCREEN, gw_mounting:70MIL_45DRILL_NO_SILKSCREEN, F.Cu at (137.2, 121.9)
- added REF**: 70MIL_45DRILL_NO_SILKSCREEN, gw_mounting:70MIL_45DRILL_NO_SILKSCREEN, F.Cu at (167.6, 106.7)
- added REF**: 70MIL_45DRILL_NO_SILKSCREEN, gw_mounting:70MIL_45DRILL_NO_SILKSCREEN, F.Cu at (96.5, 142.2)
- added REF**: 70MIL_45DRILL_NO_SILKSCREEN, gw_mounting:70MIL_45DRILL_NO_SILKSCREEN, F.Cu at (167.6, 116.8)
- added REF**: 70MIL_45DRILL_NO_SILKSCREEN, gw_mounting:70MIL_45DRILL_NO_SILKSCREEN, F.Cu at (167.6, 86.4)
- added REF**: 70MIL_45DRILL_NO_SILKSCREEN, gw_mounting:70MIL_45DRILL_NO_SILKSCREEN, F.Cu at (167.6, 96.5)
- added REF**: 70MIL_45DRILL_NO_SILKSCREEN, gw_mounting:70MIL_45DRILL_NO_SILKSCREEN, F.Cu at (167.6, 91.4)
- added REF**: 70MIL_45DRILL_NO_SILKSCREEN, gw_mounting:70MIL_45DRILL_NO_SILKSCREEN, F.Cu at (170.2, 91.4)
- added REF**: 70MIL_45DRILL_NO_SILKSCREEN, gw_mounting:70MIL_45DRILL_NO_SILKSCREEN, F.Cu at (170.2, 88.9)
- added REF**: 70MIL_45DRILL_NO_SILKSCREEN, gw_mounting:70MIL_45DRILL_NO_SILKSCREEN, F.Cu at (170.2, 86.4)
- added REF**: 70MIL_45DRILL_NO_SILKSCREEN, gw_mounting:70MIL_45DRILL_NO_SILKSCREEN, F.Cu at (167.6, 88.9)
- added REF**: 70MIL_45DRILL_NO_SILKSCREEN, gw_mounting:70MIL_45DRILL_NO_SILKSCREEN, F.Cu at (170.2, 94.0)
- added REF**: 70MIL_45DRILL_NO_SILKSCREEN, gw_mounting:70MIL_45DRILL_NO_SILKSCREEN, F.Cu at (175.3, 111.8)
- added REF**: 70MIL_45DRILL_NO_SILKSCREEN, gw_mounting:70MIL_45DRILL_NO_SILKSCREEN, F.Cu at (88.9, 139.7)
- added REF**: 70MIL_45DRILL_NO_SILKSCREEN, gw_mounting:70MIL_45DRILL_NO_SILKSCREEN, F.Cu at (172.7, 109.2)
- added REF**: 70MIL_45DRILL_NO_SILKSCREEN, gw_mounting:70MIL_45DRILL_NO_SILKSCREEN, F.Cu at (175.3, 109.2)
- added REF**: 70MIL_45DRILL_NO_SILKSCREEN, gw_mounting:70MIL_45DRILL_NO_SILKSCREEN, F.Cu at (172.7, 111.8)
- added REF**: 70MIL_45DRILL_NO_SILKSCREEN, gw_mounting:70MIL_45DRILL_NO_SILKSCREEN, F.Cu at (175.3, 116.8)
- added REF**: 70MIL_45DRILL_NO_SILKSCREEN, gw_mounting:70MIL_45DRILL_NO_SILKSCREEN, F.Cu at (172.7, 114.3)
- added REF**: 70MIL_45DRILL_NO_SILKSCREEN, gw_mounting:70MIL_45DRILL_NO_SILKSCREEN, F.Cu at (175.3, 114.3)
- added REF**: 70MIL_45DRILL_NO_SILKSCREEN, gw_mounting:70MIL_45DRILL_NO_SILKSCREEN, F.Cu at (175.3, 121.9)
- added REF**: 70MIL_45DRILL_NO_SILKSCREEN, gw_mounting:70MIL_45DRILL_NO_SILKSCREEN, F.Cu at (172.7, 119.4)
- added REF**: 70MIL_45DRILL_NO_SILKSCREEN, gw_mounting:70MIL_45DRILL_NO_SILKSCREEN, F.Cu at (175.3, 119.4)
- added REF**: 70MIL_45DRILL_NO_SILKSCREEN, gw_mounting:70MIL_45DRILL_NO_SILKSCREEN, F.Cu at (172.7, 121.9)
- added REF**: 70MIL_45DRILL_NO_SILKSCREEN, gw_mounting:70MIL_45DRILL_NO_SILKSCREEN, F.Cu at (83.8, 139.7)
- added REF**: 70MIL_45DRILL_NO_SILKSCREEN, gw_mounting:70MIL_45DRILL_NO_SILKSCREEN, F.Cu at (157.5, 86.4)
- added REF**: 70MIL_45DRILL_NO_SILKSCREEN, gw_mounting:70MIL_45DRILL_NO_SILKSCREEN, F.Cu at (157.5, 96.5)
- added REF**: 70MIL_45DRILL_NO_SILKSCREEN, gw_mounting:70MIL_45DRILL_NO_SILKSCREEN, F.Cu at (157.5, 91.4)
- added REF**: 70MIL_45DRILL_NO_SILKSCREEN, gw_mounting:70MIL_45DRILL_NO_SILKSCREEN, F.Cu at (157.5, 88.9)
- added REF**: 70MIL_45DRILL_NO_SILKSCREEN, gw_mounting:70MIL_45DRILL_NO_SILKSCREEN, F.Cu at (160.0, 94.0)
- added REF**: 70MIL_45DRILL_NO_SILKSCREEN, gw_mounting:70MIL_45DRILL_NO_SILKSCREEN, F.Cu at (165.1, 111.8)
- added REF**: 70MIL_45DRILL_NO_SILKSCREEN, gw_mounting:70MIL_45DRILL_NO_SILKSCREEN, F.Cu at (162.6, 109.2)
- added REF**: 70MIL_45DRILL_NO_SILKSCREEN, gw_mounting:70MIL_45DRILL_NO_SILKSCREEN, F.Cu at (165.1, 109.2)
- added REF**: 70MIL_45DRILL_NO_SILKSCREEN, gw_mounting:70MIL_45DRILL_NO_SILKSCREEN, F.Cu at (162.6, 111.8)
- added REF**: 70MIL_45DRILL_NO_SILKSCREEN, gw_mounting:70MIL_45DRILL_NO_SILKSCREEN, F.Cu at (165.1, 116.8)
- added REF**: 70MIL_45DRILL_NO_SILKSCREEN, gw_mounting:70MIL_45DRILL_NO_SILKSCREEN, F.Cu at (86.4, 142.2)
- added REF**: 70MIL_45DRILL_NO_SILKSCREEN, gw_mounting:70MIL_45DRILL_NO_SILKSCREEN, F.Cu at (162.6, 114.3)
- added REF**: 70MIL_45DRILL_NO_SILKSCREEN, gw_mounting:70MIL_45DRILL_NO_SILKSCREEN, F.Cu at (165.1, 114.3)
- added REF**: 70MIL_45DRILL_NO_SILKSCREEN, gw_mounting:70MIL_45DRILL_NO_SILKSCREEN, F.Cu at (165.1, 121.9)
- added REF**: 70MIL_45DRILL_NO_SILKSCREEN, gw_mounting:70MIL_45DRILL_NO_SILKSCREEN, F.Cu at (162.6, 119.4)
- added REF**: 70MIL_45DRILL_NO_SILKSCREEN, gw_mounting:70MIL_45DRILL_NO_SILKSCREEN, F.Cu at (165.1, 119.4)
- added REF**: 70MIL_45DRILL_NO_SILKSCREEN, gw_mounting:70MIL_45DRILL_NO_SILKSCREEN, F.Cu at (162.6, 121.9)
- added REF**: 70MIL_45DRILL_NO_SILKSCREEN, gw_mounting:70MIL_45DRILL_NO_SILKSCREEN, F.Cu at (160.0, 114.3)
- added REF**: 70MIL_45DRILL_NO_SILKSCREEN, gw_mounting:70MIL_45DRILL_NO_SILKSCREEN, F.Cu at (160.0, 121.9)
- added REF**: 70MIL_45DRILL_NO_SILKSCREEN, gw_mounting:70MIL_45DRILL_NO_SILKSCREEN, F.Cu at (157.5, 119.4)
- added REF**: 70MIL_45DRILL_NO_SILKSCREEN, gw_mounting:70MIL_45DRILL_NO_SILKSCREEN, F.Cu at (165.1, 106.7)
- added REF**: 70MIL_45DRILL_NO_SILKSCREEN, gw_mounting:70MIL_45DRILL_NO_SILKSCREEN, F.Cu at (83.8, 144.8)
- added REF**: 70MIL_45DRILL_NO_SILKSCREEN, gw_mounting:70MIL_45DRILL_NO_SILKSCREEN, F.Cu at (162.6, 104.1)
- added REF**: 70MIL_45DRILL_NO_SILKSCREEN, gw_mounting:70MIL_45DRILL_NO_SILKSCREEN, F.Cu at (160.0, 91.4)
- added REF**: 70MIL_45DRILL_NO_SILKSCREEN, gw_mounting:70MIL_45DRILL_NO_SILKSCREEN, F.Cu at (160.0, 88.9)
- added REF**: 70MIL_45DRILL_NO_SILKSCREEN, gw_mounting:70MIL_45DRILL_NO_SILKSCREEN, F.Cu at (160.0, 86.4)
- added REF**: 70MIL_45DRILL_NO_SILKSCREEN, gw_mounting:70MIL_45DRILL_NO_SILKSCREEN, F.Cu at (160.0, 116.8)
- added REF**: 70MIL_45DRILL_NO_SILKSCREEN, gw_mounting:70MIL_45DRILL_NO_SILKSCREEN, F.Cu at (165.1, 104.1)
- added REF**: 70MIL_45DRILL_NO_SILKSCREEN, gw_mounting:70MIL_45DRILL_NO_SILKSCREEN, F.Cu at (160.0, 109.2)
- added REF**: 70MIL_45DRILL_NO_SILKSCREEN, gw_mounting:70MIL_45DRILL_NO_SILKSCREEN, F.Cu at (157.5, 111.8)
- added REF**: 70MIL_45DRILL_NO_SILKSCREEN, gw_mounting:70MIL_45DRILL_NO_SILKSCREEN, F.Cu at (157.5, 106.7)
- added REF**: 70MIL_45DRILL_NO_SILKSCREEN, gw_mounting:70MIL_45DRILL_NO_SILKSCREEN, F.Cu at (157.5, 116.8)
- added REF**: 70MIL_45DRILL_NO_SILKSCREEN, gw_mounting:70MIL_45DRILL_NO_SILKSCREEN, F.Cu at (195.6, 71.1)
- added REF**: 70MIL_45DRILL_NO_SILKSCREEN, gw_mounting:70MIL_45DRILL_NO_SILKSCREEN, F.Cu at (94.0, 144.8)
- added REF**: 70MIL_45DRILL_NO_SILKSCREEN, gw_mounting:70MIL_45DRILL_NO_SILKSCREEN, F.Cu at (160.0, 111.8)
- added REF**: 70MIL_45DRILL_NO_SILKSCREEN, gw_mounting:70MIL_45DRILL_NO_SILKSCREEN, F.Cu at (157.5, 109.2)
- added REF**: 70MIL_45DRILL_NO_SILKSCREEN, gw_mounting:70MIL_45DRILL_NO_SILKSCREEN, F.Cu at (157.5, 114.3)
- added REF**: 70MIL_45DRILL_NO_SILKSCREEN, gw_mounting:70MIL_45DRILL_NO_SILKSCREEN, F.Cu at (170.2, 114.3)
- added REF**: 70MIL_45DRILL_NO_SILKSCREEN, gw_mounting:70MIL_45DRILL_NO_SILKSCREEN, F.Cu at (170.2, 121.9)
- added REF**: 70MIL_45DRILL_NO_SILKSCREEN, gw_mounting:70MIL_45DRILL_NO_SILKSCREEN, F.Cu at (167.6, 119.4)
- added REF**: 70MIL_45DRILL_NO_SILKSCREEN, gw_mounting:70MIL_45DRILL_NO_SILKSCREEN, F.Cu at (162.6, 94.0)
- added REF**: 70MIL_45DRILL_NO_SILKSCREEN, gw_mounting:70MIL_45DRILL_NO_SILKSCREEN, F.Cu at (165.1, 96.5)
- added REF**: 70MIL_45DRILL_NO_SILKSCREEN, gw_mounting:70MIL_45DRILL_NO_SILKSCREEN, F.Cu at (162.6, 99.1)
- added REF**: 70MIL_45DRILL_NO_SILKSCREEN, gw_mounting:70MIL_45DRILL_NO_SILKSCREEN, F.Cu at (160.0, 81.3)
- added REF**: 70MIL_45DRILL_NO_SILKSCREEN, gw_mounting:70MIL_45DRILL_NO_SILKSCREEN, F.Cu at (94.0, 139.7)
- added REF**: 70MIL_45DRILL_NO_SILKSCREEN, gw_mounting:70MIL_45DRILL_NO_SILKSCREEN, F.Cu at (157.5, 83.8)
- added REF**: 70MIL_45DRILL_NO_SILKSCREEN, gw_mounting:70MIL_45DRILL_NO_SILKSCREEN, F.Cu at (160.0, 101.6)
- added REF**: 70MIL_45DRILL_NO_SILKSCREEN, gw_mounting:70MIL_45DRILL_NO_SILKSCREEN, F.Cu at (165.1, 83.8)
- added REF**: 70MIL_45DRILL_NO_SILKSCREEN, gw_mounting:70MIL_45DRILL_NO_SILKSCREEN, F.Cu at (165.1, 101.6)
- added REF**: 70MIL_45DRILL_NO_SILKSCREEN, gw_mounting:70MIL_45DRILL_NO_SILKSCREEN, F.Cu at (162.6, 101.6)
- added REF**: 70MIL_45DRILL_NO_SILKSCREEN, gw_mounting:70MIL_45DRILL_NO_SILKSCREEN, F.Cu at (165.1, 99.1)
- added REF**: 70MIL_45DRILL_NO_SILKSCREEN, gw_mounting:70MIL_45DRILL_NO_SILKSCREEN, F.Cu at (157.5, 81.3)
- added REF**: 70MIL_45DRILL_NO_SILKSCREEN, gw_mounting:70MIL_45DRILL_NO_SILKSCREEN, F.Cu at (157.5, 101.6)
- added REF**: 70MIL_45DRILL_NO_SILKSCREEN, gw_mounting:70MIL_45DRILL_NO_SILKSCREEN, F.Cu at (157.5, 94.0)
- added REF**: 70MIL_45DRILL_NO_SILKSCREEN, gw_mounting:70MIL_45DRILL_NO_SILKSCREEN, F.Cu at (160.0, 96.5)
- added REF**: 70MIL_45DRILL_NO_SILKSCREEN, gw_mounting:70MIL_45DRILL_NO_SILKSCREEN, F.Cu at (81.3, 142.2)
- added REF**: 70MIL_45DRILL_NO_SILKSCREEN, gw_mounting:70MIL_45DRILL_NO_SILKSCREEN, F.Cu at (157.5, 99.1)
- added REF**: 70MIL_45DRILL_NO_SILKSCREEN, gw_mounting:70MIL_45DRILL_NO_SILKSCREEN, F.Cu at (160.0, 83.8)
- added REF**: 70MIL_45DRILL_NO_SILKSCREEN, gw_mounting:70MIL_45DRILL_NO_SILKSCREEN, F.Cu at (162.6, 106.7)
- added REF**: 70MIL_45DRILL_NO_SILKSCREEN, gw_mounting:70MIL_45DRILL_NO_SILKSCREEN, F.Cu at (175.3, 106.7)
- added REF**: 70MIL_45DRILL_NO_SILKSCREEN, gw_mounting:70MIL_45DRILL_NO_SILKSCREEN, F.Cu at (172.7, 104.1)
- added REF**: 70MIL_45DRILL_NO_SILKSCREEN, gw_mounting:70MIL_45DRILL_NO_SILKSCREEN, F.Cu at (162.6, 81.3)
- added REF**: 70MIL_45DRILL_NO_SILKSCREEN, gw_mounting:70MIL_45DRILL_NO_SILKSCREEN, F.Cu at (175.3, 104.1)
- added REF**: 70MIL_45DRILL_NO_SILKSCREEN, gw_mounting:70MIL_45DRILL_NO_SILKSCREEN, F.Cu at (165.1, 86.4)
- added REF**: 70MIL_45DRILL_NO_SILKSCREEN, gw_mounting:70MIL_45DRILL_NO_SILKSCREEN, F.Cu at (165.1, 81.3)
- added REF**: 70MIL_45DRILL_NO_SILKSCREEN, gw_mounting:70MIL_45DRILL_NO_SILKSCREEN, F.Cu at (162.6, 83.8)
- added REF**: 70MIL_45DRILL_NO_SILKSCREEN, gw_mounting:70MIL_45DRILL_NO_SILKSCREEN, F.Cu at (81.3, 139.7)
- added REF**: 70MIL_45DRILL_NO_SILKSCREEN, gw_mounting:70MIL_45DRILL_NO_SILKSCREEN, F.Cu at (162.6, 96.5)
- added REF**: 70MIL_45DRILL_NO_SILKSCREEN, gw_mounting:70MIL_45DRILL_NO_SILKSCREEN, F.Cu at (160.0, 99.1)
- added REF**: 70MIL_45DRILL_NO_SILKSCREEN, gw_mounting:70MIL_45DRILL_NO_SILKSCREEN, F.Cu at (165.1, 88.9)
- added REF**: 70MIL_45DRILL_NO_SILKSCREEN, gw_mounting:70MIL_45DRILL_NO_SILKSCREEN, F.Cu at (162.6, 86.4)
- added REF**: 70MIL_45DRILL_NO_SILKSCREEN, gw_mounting:70MIL_45DRILL_NO_SILKSCREEN, F.Cu at (170.2, 111.8)
- added REF**: 70MIL_45DRILL_NO_SILKSCREEN, gw_mounting:70MIL_45DRILL_NO_SILKSCREEN, F.Cu at (167.6, 109.2)
- added REF**: 70MIL_45DRILL_NO_SILKSCREEN, gw_mounting:70MIL_45DRILL_NO_SILKSCREEN, F.Cu at (170.2, 109.2)
- added REF**: 70MIL_45DRILL_NO_SILKSCREEN, gw_mounting:70MIL_45DRILL_NO_SILKSCREEN, F.Cu at (167.6, 111.8)
- added REF**: 70MIL_45DRILL_NO_SILKSCREEN, gw_mounting:70MIL_45DRILL_NO_SILKSCREEN, F.Cu at (170.2, 116.8)
- added REF**: 70MIL_45DRILL_NO_SILKSCREEN, gw_mounting:70MIL_45DRILL_NO_SILKSCREEN, F.Cu at (167.6, 114.3)
- added REF**: 70MIL_45DRILL_NO_SILKSCREEN, gw_mounting:70MIL_45DRILL_NO_SILKSCREEN, F.Cu at (81.3, 144.8)
- added REF**: 70MIL_45DRILL_NO_SILKSCREEN, gw_mounting:70MIL_45DRILL_NO_SILKSCREEN, F.Cu at (172.7, 81.3)
- added REF**: 70MIL_45DRILL_NO_SILKSCREEN, gw_mounting:70MIL_45DRILL_NO_SILKSCREEN, F.Cu at (175.3, 81.3)
- added REF**: 70MIL_45DRILL_NO_SILKSCREEN, gw_mounting:70MIL_45DRILL_NO_SILKSCREEN, F.Cu at (172.7, 83.8)
- added REF**: 70MIL_45DRILL_NO_SILKSCREEN, gw_mounting:70MIL_45DRILL_NO_SILKSCREEN, F.Cu at (172.7, 94.0)
- added REF**: 70MIL_45DRILL_NO_SILKSCREEN, gw_mounting:70MIL_45DRILL_NO_SILKSCREEN, F.Cu at (175.3, 96.5)
- added REF**: 70MIL_45DRILL_NO_SILKSCREEN, gw_mounting:70MIL_45DRILL_NO_SILKSCREEN, F.Cu at (172.7, 99.1)
- added REF**: 70MIL_45DRILL_NO_SILKSCREEN, gw_mounting:70MIL_45DRILL_NO_SILKSCREEN, F.Cu at (170.2, 81.3)
- added REF**: 70MIL_45DRILL_NO_SILKSCREEN, gw_mounting:70MIL_45DRILL_NO_SILKSCREEN, F.Cu at (167.6, 83.8)
- added REF**: 70MIL_45DRILL_NO_SILKSCREEN, gw_mounting:70MIL_45DRILL_NO_SILKSCREEN, F.Cu at (170.2, 101.6)
- added REF**: 70MIL_45DRILL_NO_SILKSCREEN, gw_mounting:70MIL_45DRILL_NO_SILKSCREEN, F.Cu at (175.3, 83.8)
- added REF**: 70MIL_45DRILL_NO_SILKSCREEN, gw_mounting:70MIL_45DRILL_NO_SILKSCREEN, F.Cu at (94.0, 142.2)
- added REF**: 70MIL_45DRILL_NO_SILKSCREEN, gw_mounting:70MIL_45DRILL_NO_SILKSCREEN, F.Cu at (175.3, 101.6)
- added REF**: 70MIL_45DRILL_NO_SILKSCREEN, gw_mounting:70MIL_45DRILL_NO_SILKSCREEN, F.Cu at (172.7, 101.6)
- added REF**: 70MIL_45DRILL_NO_SILKSCREEN, gw_mounting:70MIL_45DRILL_NO_SILKSCREEN, F.Cu at (175.3, 99.1)
- added REF**: 70MIL_45DRILL_NO_SILKSCREEN, gw_mounting:70MIL_45DRILL_NO_SILKSCREEN, F.Cu at (167.6, 81.3)
- added REF**: 70MIL_45DRILL_NO_SILKSCREEN, gw_mounting:70MIL_45DRILL_NO_SILKSCREEN, F.Cu at (160.0, 106.7)
- added REF**: 70MIL_45DRILL_NO_SILKSCREEN, gw_mounting:70MIL_45DRILL_NO_SILKSCREEN, F.Cu at (157.5, 104.1)
- added REF**: 70MIL_45DRILL_NO_SILKSCREEN, gw_mounting:70MIL_45DRILL_NO_SILKSCREEN, F.Cu at (160.0, 104.1)
- added REF**: 70MIL_45DRILL_NO_SILKSCREEN, gw_mounting:70MIL_45DRILL_NO_SILKSCREEN, F.Cu at (162.6, 116.8)
- added REF**: 70MIL_45DRILL_NO_SILKSCREEN, gw_mounting:70MIL_45DRILL_NO_SILKSCREEN, F.Cu at (167.6, 101.6)
- added REF**: 70MIL_45DRILL_NO_SILKSCREEN, gw_mounting:70MIL_45DRILL_NO_SILKSCREEN, F.Cu at (167.6, 94.0)
- added REF**: 70MIL_45DRILL_NO_SILKSCREEN, gw_mounting:70MIL_45DRILL_NO_SILKSCREEN, F.Cu at (96.5, 139.7)
- added REF**: 70MIL_45DRILL_NO_SILKSCREEN, gw_mounting:70MIL_45DRILL_NO_SILKSCREEN, F.Cu at (170.2, 96.5)
- added REF**: 70MIL_45DRILL_NO_SILKSCREEN, gw_mounting:70MIL_45DRILL_NO_SILKSCREEN, F.Cu at (167.6, 99.1)
- added REF**: 70MIL_45DRILL_NO_SILKSCREEN, gw_mounting:70MIL_45DRILL_NO_SILKSCREEN, F.Cu at (170.2, 83.8)
- added REF**: 70MIL_45DRILL_NO_SILKSCREEN, gw_mounting:70MIL_45DRILL_NO_SILKSCREEN, F.Cu at (172.7, 106.7)
- added REF**: 70MIL_45DRILL_NO_SILKSCREEN, gw_mounting:70MIL_45DRILL_NO_SILKSCREEN, F.Cu at (172.7, 96.5)
- added REF**: 70MIL_45DRILL_NO_SILKSCREEN, gw_mounting:70MIL_45DRILL_NO_SILKSCREEN, F.Cu at (170.2, 99.1)
- added REF**: 70MIL_45DRILL_NO_SILKSCREEN, gw_mounting:70MIL_45DRILL_NO_SILKSCREEN, F.Cu at (175.3, 88.9)
- added REF**: 70MIL_45DRILL_NO_SILKSCREEN, gw_mounting:70MIL_45DRILL_NO_SILKSCREEN, F.Cu at (172.7, 86.4)
- added REF**: 70MIL_45DRILL_NO_SILKSCREEN, gw_mounting:70MIL_45DRILL_NO_SILKSCREEN, F.Cu at (175.3, 86.4)
- added REF**: 70MIL_45DRILL_NO_SILKSCREEN, gw_mounting:70MIL_45DRILL_NO_SILKSCREEN, F.Cu at (172.7, 88.9)
- added REF**: 70MIL_45DRILL_NO_SILKSCREEN, gw_mounting:70MIL_45DRILL_NO_SILKSCREEN, F.Cu at (86.4, 139.7)
- added REF**: 70MIL_45DRILL_NO_SILKSCREEN, gw_mounting:70MIL_45DRILL_NO_SILKSCREEN, F.Cu at (175.3, 94.0)
- added REF**: 70MIL_45DRILL_NO_SILKSCREEN, gw_mounting:70MIL_45DRILL_NO_SILKSCREEN, F.Cu at (172.7, 91.4)
- added REF**: 70MIL_45DRILL_NO_SILKSCREEN, gw_mounting:70MIL_45DRILL_NO_SILKSCREEN, F.Cu at (175.3, 91.4)
- added REF**: 70MIL_45DRILL_NO_SILKSCREEN, gw_mounting:70MIL_45DRILL_NO_SILKSCREEN, F.Cu at (170.2, 119.4)
- added REF**: 70MIL_45DRILL_NO_SILKSCREEN, gw_mounting:70MIL_45DRILL_NO_SILKSCREEN, F.Cu at (167.6, 121.9)
- added REF**: 70MIL_45DRILL_NO_SILKSCREEN, gw_mounting:70MIL_45DRILL_NO_SILKSCREEN, F.Cu at (170.2, 106.7)
- added REF**: 70MIL_45DRILL_NO_SILKSCREEN, gw_mounting:70MIL_45DRILL_NO_SILKSCREEN, F.Cu at (167.6, 104.1)
- added REF**: 70MIL_45DRILL_NO_SILKSCREEN, gw_mounting:70MIL_45DRILL_NO_SILKSCREEN, F.Cu at (170.2, 104.1)
- added REF**: 70MIL_45DRILL_NO_SILKSCREEN, gw_mounting:70MIL_45DRILL_NO_SILKSCREEN, F.Cu at (172.7, 116.8)
- added REF**: 70MIL_45DRILL_NO_SILKSCREEN, gw_mounting:70MIL_45DRILL_NO_SILKSCREEN, F.Cu at (162.6, 88.9)
- added REF**: 70MIL_45DRILL_NO_SILKSCREEN, gw_mounting:70MIL_45DRILL_NO_SILKSCREEN, F.Cu at (91.4, 137.2)
- added REF**: 70MIL_45DRILL_NO_SILKSCREEN, gw_mounting:70MIL_45DRILL_NO_SILKSCREEN, F.Cu at (165.1, 94.0)
- added REF**: 70MIL_45DRILL_NO_SILKSCREEN, gw_mounting:70MIL_45DRILL_NO_SILKSCREEN, F.Cu at (162.6, 91.4)
- added REF**: 70MIL_45DRILL_NO_SILKSCREEN, gw_mounting:70MIL_45DRILL_NO_SILKSCREEN, F.Cu at (160.0, 119.4)
- added REF**: 70MIL_45DRILL_NO_SILKSCREEN, gw_mounting:70MIL_45DRILL_NO_SILKSCREEN, F.Cu at (165.1, 91.4)
- added REF**: 70MIL_45DRILL_NO_SILKSCREEN, gw_mounting:70MIL_45DRILL_NO_SILKSCREEN, F.Cu at (157.5, 121.9)
- added REF**: 70MIL_45DRILL_NO_SILKSCREEN, gw_mounting:70MIL_45DRILL_NO_SILKSCREEN, F.Cu at (177.8, 106.7)
- added REF**: 70MIL_45DRILL_NO_SILKSCREEN, gw_mounting:70MIL_45DRILL_NO_SILKSCREEN, F.Cu at (177.8, 116.8)
- added REF**: 70MIL_45DRILL_NO_SILKSCREEN, gw_mounting:70MIL_45DRILL_NO_SILKSCREEN, F.Cu at (177.8, 86.4)
- added REF**: 70MIL_45DRILL_NO_SILKSCREEN, gw_mounting:70MIL_45DRILL_NO_SILKSCREEN, F.Cu at (177.8, 96.5)
- added REF**: 70MIL_45DRILL_NO_SILKSCREEN, gw_mounting:70MIL_45DRILL_NO_SILKSCREEN, F.Cu at (177.8, 91.4)
- added REF**: 70MIL_45DRILL_NO_SILKSCREEN, gw_mounting:70MIL_45DRILL_NO_SILKSCREEN, F.Cu at (88.9, 134.6)
- added REF**: 70MIL_45DRILL_NO_SILKSCREEN, gw_mounting:70MIL_45DRILL_NO_SILKSCREEN, F.Cu at (180.3, 91.4)
- added REF**: 70MIL_45DRILL_NO_SILKSCREEN, gw_mounting:70MIL_45DRILL_NO_SILKSCREEN, F.Cu at (180.3, 88.9)
- added REF**: 70MIL_45DRILL_NO_SILKSCREEN, gw_mounting:70MIL_45DRILL_NO_SILKSCREEN, F.Cu at (180.3, 86.4)
- added REF**: 70MIL_45DRILL_NO_SILKSCREEN, gw_mounting:70MIL_45DRILL_NO_SILKSCREEN, F.Cu at (177.8, 88.9)
- added REF**: 70MIL_45DRILL_NO_SILKSCREEN, gw_mounting:70MIL_45DRILL_NO_SILKSCREEN, F.Cu at (180.3, 94.0)
- added REF**: 70MIL_45DRILL_NO_SILKSCREEN, gw_mounting:70MIL_45DRILL_NO_SILKSCREEN, F.Cu at (185.4, 111.8)
- added REF**: 70MIL_45DRILL_NO_SILKSCREEN, gw_mounting:70MIL_45DRILL_NO_SILKSCREEN, F.Cu at (182.9, 109.2)
- added REF**: 70MIL_45DRILL_NO_SILKSCREEN, gw_mounting:70MIL_45DRILL_NO_SILKSCREEN, F.Cu at (185.4, 109.2)
- added REF**: 70MIL_45DRILL_NO_SILKSCREEN, gw_mounting:70MIL_45DRILL_NO_SILKSCREEN, F.Cu at (182.9, 111.8)
- added REF**: 70MIL_45DRILL_NO_SILKSCREEN, gw_mounting:70MIL_45DRILL_NO_SILKSCREEN, F.Cu at (185.4, 116.8)
- added REF**: 70MIL_45DRILL_NO_SILKSCREEN, gw_mounting:70MIL_45DRILL_NO_SILKSCREEN, F.Cu at (193.0, 68.6)
- added REF**: 70MIL_45DRILL_NO_SILKSCREEN, gw_mounting:70MIL_45DRILL_NO_SILKSCREEN, F.Cu at (91.4, 134.6)
- added REF**: 70MIL_45DRILL_NO_SILKSCREEN, gw_mounting:70MIL_45DRILL_NO_SILKSCREEN, F.Cu at (182.9, 114.3)
- added REF**: 70MIL_45DRILL_NO_SILKSCREEN, gw_mounting:70MIL_45DRILL_NO_SILKSCREEN, F.Cu at (185.4, 114.3)
- added REF**: 70MIL_45DRILL_NO_SILKSCREEN, gw_mounting:70MIL_45DRILL_NO_SILKSCREEN, F.Cu at (185.4, 121.9)
- added REF**: 70MIL_45DRILL_NO_SILKSCREEN, gw_mounting:70MIL_45DRILL_NO_SILKSCREEN, F.Cu at (182.9, 119.4)
- added REF**: 70MIL_45DRILL_NO_SILKSCREEN, gw_mounting:70MIL_45DRILL_NO_SILKSCREEN, F.Cu at (185.4, 119.4)
- added REF**: 70MIL_45DRILL_NO_SILKSCREEN, gw_mounting:70MIL_45DRILL_NO_SILKSCREEN, F.Cu at (182.9, 121.9)
- added REF**: 70MIL_45DRILL_NO_SILKSCREEN, gw_mounting:70MIL_45DRILL_NO_SILKSCREEN, F.Cu at (180.3, 114.3)
- added REF**: 70MIL_45DRILL_NO_SILKSCREEN, gw_mounting:70MIL_45DRILL_NO_SILKSCREEN, F.Cu at (180.3, 121.9)
- added REF**: 70MIL_45DRILL_NO_SILKSCREEN, gw_mounting:70MIL_45DRILL_NO_SILKSCREEN, F.Cu at (177.8, 119.4)
- added REF**: 70MIL_45DRILL_NO_SILKSCREEN, gw_mounting:70MIL_45DRILL_NO_SILKSCREEN, F.Cu at (185.4, 106.7)
- added REF**: 70MIL_45DRILL_NO_SILKSCREEN, gw_mounting:70MIL_45DRILL_NO_SILKSCREEN, F.Cu at (88.9, 137.2)
- added REF**: 70MIL_45DRILL_NO_SILKSCREEN, gw_mounting:70MIL_45DRILL_NO_SILKSCREEN, F.Cu at (182.9, 104.1)
- added REF**: 70MIL_45DRILL_NO_SILKSCREEN, gw_mounting:70MIL_45DRILL_NO_SILKSCREEN, F.Cu at (185.4, 104.1)
- added REF**: 70MIL_45DRILL_NO_SILKSCREEN, gw_mounting:70MIL_45DRILL_NO_SILKSCREEN, F.Cu at (180.3, 111.8)
- added REF**: 70MIL_45DRILL_NO_SILKSCREEN, gw_mounting:70MIL_45DRILL_NO_SILKSCREEN, F.Cu at (177.8, 109.2)
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Connections:
- J2 pad 1: (no net) -> PD7
- J2 pad 2: (no net) -> PD6
- J2 pad 3: (no net) -> PD5
- J2 pad 4: (no net) -> PD4
- J2 pad 5: (no net) -> PD3
- J2 pad 6: (no net) -> PD2
- J2 pad 7: (no net) -> PD1
- J2 pad 8: (no net) -> PD0
- J3 pad 1: (no net) -> PB0
- J3 pad 2: (no net) -> PB1
- J3 pad 3: (no net) -> PB2
- J3 pad 4: (no net) -> PB3
- J3 pad 5: (no net) -> PB4
- J3 pad 6: (no net) -> PB5
- J3 pad 7: (no net) -> PB6
- J3 pad 8: (no net) -> PB7
- J5 pad 10: (no net) -> BA7
- J5 pad 11: (no net) -> BA8
- J5 pad 12: (no net) -> BA9
- J5 pad 13: (no net) -> BA10
- J5 pad 14: (no net) -> BA11
- J5 pad 15: (no net) -> BA12
- J5 pad 16: (no net) -> BA13
- J5 pad 17: (no net) -> BA14
- J5 pad 18: (no net) -> BA15
- J5 pad 21: (no net) -> *BMASK
- J5 pad 22: (no net) -> BCLOCK
- J5 pad 23: (no net) -> *BSTART
- J5 pad 25: (no net) -> BIO**M
- J5 pad 26: (no net) -> *BRESET
- J5 pad 27: (no net) -> BR**W
- J5 pad 28: (no net) -> *BINT
- J5 pad 29: GND -> *BSELECTED
- J5 pad 3: (no net) -> BA0
- J5 pad 30: (no net) -> BREADY
- J5 pad 31: (no net) -> BD0
- J5 pad 32: (no net) -> BD1
- J5 pad 33: (no net) -> BD2
- J5 pad 34: (no net) -> BD3
- J5 pad 35: (no net) -> BD4
- J5 pad 36: (no net) -> BD5
- J5 pad 37: (no net) -> BD6
- J5 pad 38: (no net) -> BD7
- J5 pad 4: (no net) -> BA1
- J5 pad 5: (no net) -> BA2
- J5 pad 6: (no net) -> BA3
- J5 pad 7: (no net) -> BA4
- J5 pad 8: (no net) -> BA5
- J5 pad 9: (no net) -> BA6
Routing:
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Other:
- board text added: "*BINT"
- board text added: "*BMASK"
- board text added: "*BRESET"
- board text added: "*BSEL’D"
- board text added: "*BSTART"
- board text added: "BA0"
- board text added: "BA1"
- board text added: "BA10"
- board text added: "BA11"
- board text added: "BA12"
- board text added: "BA13"
- board text added: "BA14"
- board text added: "BA15"
- board text added: "BA2"
- board text added: "BA3"
- board text added: "BA4"
- board text added: "BA5"
- board text added: "BA6"
- board text added: "BA7"
- board text added: "BA8"
- board text added: "BA9"
- board text added: "BCLOCK"
- board text added: "BD0"
- board text added: "BD1"
- board text added: "BD2"
- board text added: "BD3"
- board text added: "BD4"
- board text added: "BD5"
- board text added: "BD6"
- board text added: "BD7"
- board text added: "BIO**M"
- board text added: "BR**W"
- board text added: "BREADY"
- board text added: "GW-R65X1Q-PROTO1"
- board text added: "PB0"
- board text added: "PB1"
- board text added: "PB2"
- board text added: "PB3"
- board text added: "PB4"
- board text added: "PB5"
- board text added: "PB6"
- board text added: "PB7"
- board text added: "PD0"
- board text added: "PD1"
- board text added: "PD2"
- board text added: "PD3"
- board text added: "PD4"
- board text added: "PD5"
- board text added: "PD6"
- board text added: "PD7"
- board text added: "PORT B"
- board text added: "PORT D"
- board text added: "R65X1Q SBC PROTOTYPING BOARD http://www.glitchwrks.com"
- board text removed: "GW-R65X1QSBC-PROTO1"
- board text removed: "http://www.glitchwrks.com/"
