File: gw-r65x1qsbc-proto1.sch (KiCad schematic (older format))
At the start: 8 parts, among them J2 PORT D, J3 PORT B, J5 GLITCHBUS

Commit message: PROTOTYPE 1
Parts:
- added J1: PORT D, gw_headers:STRAIGHT_2x5_NOSILK, symbol gw_computer_busses:R65X1QSBC_PORTD
- added J4: PORT B, gw_headers:STRAIGHT_2x5, symbol gw_computer_busses:R65X1QSBC_PORTB
- added J6: GLITCHBUS, gw_headers:STRAIGHT_2x20, symbol gw_computer_busses:GLITCHBUS_1.0
- J3: footprint gw_headers:STRAIGHT_2x5 -> gw_headers:STRAIGHT_2x5_NOSILK
- J5: footprint gw_headers:STRAIGHT_2x20 -> gw_headers:STRAIGHT_2x20_NOSILK; symbol gw_computer_busses:GLITCHBUS -> gw_computer_busses:GLITCHBUS_1.0
Connections:
- net *BINT: now also J6.28 (*BINT)
- net *BMASK: now also J6.21 (*BMASK)
- net *BRESET: now also J6.26 (*BRESET)
- net *BSTART: now also J6.23 (*BSTART)
- net BA0: now also J6.3 (BA0)
- net BA1: now also J6.4 (BA1)
- net BA10: now also J6.13 (BA10)
- net BA11: now also J6.14 (BA11)
- net BA12: now also J6.15 (BA12)
- net BA13: now also J6.16 (BA13)
- net BA14: now also J6.17 (BA14)
- net BA15: now also J6.18 (BA15)
- net BA2: now also J6.5 (BA2)
- net BA3: now also J6.6 (BA3)
- net BA4: now also J6.7 (BA4)
- net BA5: now also J6.8 (BA5)
- net BA6: now also J6.9 (BA6)
- net BA7: now also J6.10 (BA7)
- net BA8: now also J6.11 (BA8)
- net BA9: now also J6.12 (BA9)
- net BCLOCK: now also J6.22 (BCLOCK)
- net BD0: now also J6.31 (BD0)
- net BD1: now also J6.32 (BD1)
- net BD2: now also J6.33 (BD2)
- net BD3: now also J6.34 (BD3)
- net BD4: now also J6.35 (BD4)
- net BD5: now also J6.36 (BD5)
- net BD6: now also J6.37 (BD6)
- net BD7: now also J6.38 (BD7)
- net BIO**M: now also J6.25 (BIO**M)
- net BR**W: now also J6.27 (BR**W)
- net BREADY: now also J6.30 (BREADY)
- net GND: now also J1.10 (GND), J1.9 (GND), J4.10 (GND), J4.9 (GND), J6.19 (GND), J6.20 (GND), J6.24 (GND), J6.39 (GND), J6.40 (GND); no longer J5.29 (GND)
- net PB0: now also J4.1 (PB0)
- net PB1: now also J4.2 (PB1)
- net PB2: now also J4.3 (PB2)
- net PB3: now also J4.4 (PB3)
- net PB4: now also J4.5 (PB4)
- net PB5: now also J4.6 (PB5)
- net PB6: now also J4.7 (PB6)
- net PB7: now also J4.8 (PB7)
- net PD0: now also J1.8 (PD0)
- net PD1: now also J1.7 (PD1)
- net PD2: now also J1.6 (PD2)
- net PD3: now also J1.5 (PD3)
- net PD4: now also J1.4 (PD4)
- net PD5: now also J1.3 (PD5)
- net PD6: now also J1.2 (PD6)
- net PD7: now also J1.1 (PD7)
- net VCC: now also J6.1 (VCC), J6.2 (VCC)
- new net *BSELECTED: J5.29 (*BSELECTED), J6.29 (*BSELECTED)
